File: counter.kicad_pcb (KiCad board)
At the start: 2 copper layers, 60 x 100 mm, 42 parts, among them J1 Eurorack Power, J2 Clock In 1, J3 Reset In 1, J4 Clock In 2, J5 Reset In 2, Q1 2N3904, Q2 2N3904, SW1 Reset 1, SW2 Reset 2, U1 LM7805_TO220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

Commit message: Rev. 2
Parts:
- added H1: MountingHole, MountingHole:MountingHole_4.3mm_M4, B.Cu at (125.4, 53.3)
- C1: footprint Capacitor_THT:CP_Radial_D6.3mm_P2.50mm -> Capacitor_THT:CP_Radial_D5.0mm_P2.00mm
- R1, R6: value 1k -> 10k
- moved REF** 30.8 mm to (109.9, 134.3)
- moved R5 12.1 mm to (109.5, 118.4), turned to -90 degrees
- moved R4 9.16 mm to (97.8, 113.7), turned to 0 degrees
- moved D4 6.83 mm to (84.8, 113.8)
- moved R1 6.35 mm to (110.5, 113.7)
- moved C2 5.50 mm to (79.1, 114.0)
- moved D3 5.08 mm to (93.3, 116.8)
- moved C1 4.90 mm to (83.8, 130.4)
- moved J1 4.90 mm to (74.9, 128.4)
- moved J2 4.90 mm to (118.1, 122.2)
- moved J3 4.90 mm to (101.6, 122.2)
- moved R10 4.90 mm to (93.2, 142.4)
- moved R6 4.90 mm to (114.3, 130.4)
- moved R9 4.90 mm to (105.4, 130.4)
- moved SW1 4.90 mm to (85.1, 122.2)
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Routing:
- net Net-(J2-PadT): track 56.6 -> 35.9 mm
- net RST2: track 104.1 -> 88.4 mm, vias 1 -> 0
- net +5V: track 255.8 -> 241.5 mm, vias 5 -> 4
- net CLK2: track 75.2 -> 70.5 mm
- net Net-(D4-K): track 7.61 -> 12.0 mm
- net RST1: track 109.7 -> 113.9 mm
- net Net-(Q1-B): track 12.5 -> 15.7 mm
- net Net-(U2B-~{CP0}): track 109.3 -> 112.1 mm
- net CLK1: track 66.0 -> 64.2 mm
- net Net-(D3-K): track 4.49 -> 3.65 mm
- net Net-(D3-A): track 24.3 -> 25.0 mm
Other:
- board size 60 x 100 mm -> 60 x 98.1 mm
- board text added: "Counter rev. 2 March 22, 2026"
- board text removed: "Counter rev. 1 Sept 27, 2025"
